File: nes_keyboard.kicad_pcb (KiCad board)
At the start: 2 copper layers, 323.9 x 115.5 mm, 257 parts, among them J1 USB_C_Receptacle_USB2.0_16P, J2 Conn_01x02_Pin, SW1 SW_Push, SW2 SW_Push, SW3 RotaryEncoder_Switch_MP, U1 RP2040, U2 W25Q128JVS, U4 74AHCT1G125, Y1 Crystal_GND24

Commit message: PCB Modifications (all) - V0.2
Parts:
- moved C15 9.26 mm to (53.6, 57.1)
Routing:
- net Net-(D87-DOUT): track 19.1 -> 21.5 mm
- net Net-(D86-DOUT): track 19.1 -> 21.4 mm
- net +5V: track 2.62 -> 3.97 mm, vias 15 -> 13
- net GND: vias 268 -> 253
