File: nes_keyboard.kicad_pcb (KiCad board)
At the start: 2 copper layers, 323.9 x 115.5 mm, 257 parts, among them J1 USB_C_Receptacle_USB2.0_16P, J2 Conn_01x02_Pin, SW1 SW_Push, SW2 SW_Push, SW3 RotaryEncoder_Switch_MP, U1 RP2040, U2 W25Q128JVS, U4 74AHCT1G125, Y1 Crystal_GND24

Commit message: Updated main board + daughterboard layout - V0.3
Parts:
- removed J2: Conn_01x02_Pin, Connector_Hirose:Hirose_DF13-02P-1.25DS_1x02_P1.25mm_Horizontal
- removed REF** (x3): Stabilizer_MX_2.00u, ScottoKeebs_Stabilizer:Stabilizer_MX_2.00u
- removed REF**: Stabilizer_MX_6.25u, ScottoKeebs_Stabilizer:Stabilizer_MX_6.25u
- removed TP17, TP18: TestPoint, TestPoint:TestPoint_Pad_D1.0mm
- added C23: 10uF, Capacitor_SMD:C_0805_2012Metric, B.Cu at (63.6, 140.7)
- added C24: 10uF, Capacitor_SMD:C_0805_2012Metric, B.Cu at (70.3, 132.5)
- added S85: Keyswitch, PCM_Mounting_Keyboard_Stabilizer:Stabilizer_Cherry_MX_2.00u, F.Cu at (335.8, 61.5)
- added S86: Keyswitch, PCM_Mounting_Keyboard_Stabilizer:Stabilizer_Cherry_MX_2.00u, F.Cu at (333.4, 99.7)
- added S87: Keyswitch, PCM_Mounting_Keyboard_Stabilizer:Stabilizer_Cherry_MX_2.00u, F.Cu at (90.5, 118.7)
- added S88: Keyswitch, PCM_Mounting_Keyboard_Stabilizer:Stabilizer_Cherry_MX_6.25u, F.Cu at (200.0, 137.8)
- added U3: W25Q128JVE, Package_SON:WSON-8-1EP_8x6mm_P1.27mm_EP3.4x4.3mm, B.Cu at (62.2, 116.9)
- C1, C11, C12, C16, C25, C26, C27, C28, C29: footprint Capacitor_SMD:C_0402_1005Metric_Pad0.74x0.62mm_HandSolder -> Capacitor_SMD:C_0402_1005Metric
- C10, C13, C14, C2, C3, C4, C5, C6, C7, C8, C9: value 100nF -> 0.1uF; footprint Capacitor_SMD:C_0402_1005Metric_Pad0.74x0.62mm_HandSolder -> Capacitor_SMD:C_0402_1005Metric
- C15: footprint Capacitor_SMD:C_0603_1608Metric_Pad1.08x0.95mm_HandSolder -> Capacitor_SMD:C_0805_2012Metric
- C17, C18, C19, C20, C21, C22: footprint Capacitor_SMD:C_0603_1608Metric_Pad1.08x0.95mm_HandSolder -> Capacitor_SMD:C_0603_1608Metric
- R1, R13, R2, R4, R5, R8: footprint Resistor_SMD:R_0603_1608Metric_Pad0.98x0.95mm_HandSolder -> Resistor_SMD:R_0603_1608Metric
- R10, R11, R12, R7, R9: footprint Resistor_SMD:R_0402_1005Metric_Pad0.72x0.64mm_HandSolder -> Resistor_SMD:R_0402_1005Metric
- R3: footprint Resistor_SMD:R_0603_1608Metric_Pad0.98x0.95mm_HandSolder -> Resistor_SMD:R_0402_1005Metric
- TP1, TP2, TP3, TP4: moved to F.Cu
- U1: footprint Package_DFN_QFN:QFN-56-1EP_7x7mm_P0.4mm_EP3.2x3.2mm -> Package_DFN_QFN:QFN-56-1EP_7x7mm_P0.4mm_EP3.2x3.2mm_ThermalVias
- U2: value W25Q128JVS -> NCP1117-3.3_SOT223; footprint Package_SO:SOIC-8_5.3x5.3mm_P1.27mm -> Package_TO_SOT_SMD:SOT-223-3_TabPin2
- Y1: footprint Crystal:Crystal_SMD_3225-4Pin_3.2x2.5mm_HandSoldering -> Crystal:Crystal_SMD_3225-4Pin_3.2x2.5mm
- moved F1 146.7 mm to (67.7, 131.8), turned to 90 degrees
- moved R5 132.0 mm to (58.1, 116.4), turned to 90 degrees
- moved SW1 131.0 mm to (57.5, 124.8)
- moved R4 126.5 mm to (58.1, 113.2), turned to -90 degrees
- moved C13 123.3 mm to (60.2, 122.7), turned to -90 degrees
- moved U2 117.3 mm to (68.4, 138.0), turned to 90 degrees
- moved C4 115.8 mm to (63.5, 110.0), turned to -90 degrees
- moved R1 115.2 mm to (68.8, 117.5), turned to 90 degrees
- moved C3 114.5 mm to (66.7, 112.9), turned to -90 degrees
- moved C10 114.0 mm to (62.0, 103.9), turned to 135 degrees
- moved R2 113.6 mm to (70.3, 117.5), turned to -90 degrees
- moved C7 113.2 mm to (67.8, 112.9), turned to -90 degrees
- moved TP16 110.7 mm to (60.6, 128.8), turned to 0 degrees
- moved C16 108.4 mm to (70.9, 112.3), turned to -90 degrees
- moved C1 107.1 mm to (72.0, 112.3), turned to -90 degrees
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Connections:
- net /MCU/EN renamed Net-(U1-RUN)
- C15 pad 1: +5V -> VBUS
- C17 pad 1: +5V -> VBUS
- C18 pad 1: +5V -> VBUS
- C19 pad 1: +5V -> VBUS
- C20 pad 1: +5V -> VBUS
- C21 pad 1: +5V -> VBUS
- C22 pad 1: +5V -> VBUS
- C29 pad 1: +5V -> VBUS
- D85 pad 1: +5V -> VBUS
- D86 pad 1: +5V -> VBUS
- D87 pad 1: +5V -> VBUS
- D88 pad 1: +5V -> VBUS
- D89 pad 1: +5V -> VBUS
- D90 pad 1: +5V -> VBUS
- J1 pad A4: VDD -> VBUS
- J1 pad A5: unconnected-(J1-CC1-PadA5) -> VDD
- J1 pad A9: VDD -> VBUS
- J1 pad B4: VDD -> VBUS
- J1 pad B5: unconnected-(J1-CC2-PadB5) -> VDD
- J1 pad B9: VDD -> VBUS
- TP2 pad 1: /MCU/SWCLK -> /MCU/SWD
- TP3 pad 1: /MCU/SWD -> /MCU/SWCLK
- U1 pad 11: /C14 -> /C15
- U1 pad 12: /C15 -> /C14
- U1 pad 13: /C16 -> /C12
- U1 pad 14: /C1 -> /C11
- U1 pad 15: /C2 -> /C10
- U1 pad 16: /C3 -> /C9
- U1 pad 17: /C4 -> /C8
- U1 pad 18: /C5 -> /R4
- U1 pad 2: /C6 -> /LED_DATA
- U1 pad 27: /R1 -> /C7
- U1 pad 28: /R2 -> /C6
- U1 pad 29: /R6 -> /C5
- U1 pad 3: /C7 -> /TERMINAL_B
- U1 pad 30: /R5 -> /C4
- U1 pad 31: /R4 -> /C3
- U1 pad 32: /R3 -> /C2
- U1 pad 34: /LED_DATA -> /C1
- U1 pad 35: /TERMINAL_B -> /R3
- U1 pad 36: /TERMINAL_A -> /R2
- U1 pad 37: /SW -> /R1
- U1 pad 4: /C8 -> /TERMINAL_A
- U1 pad 5: /C9 -> /SW
- U1 pad 6: /C10 -> /R6
- U1 pad 7: /C11 -> /R5
- U1 pad 8: /C12 -> /C13
- U1 pad 9: /C13 -> /C16
- U2 pad 1: /MCU/QSPI_SS -> GND
- U2 pad 2: /MCU/QSPI_SD1 -> VDD
- U2 pad 3: /MCU/QSPI_SD2 -> VBUS
- U4 pad 5: +5V -> VBUS
Routing:
- net +3V3: track 345.6 -> 165.7 mm, vias 28 -> 9
- net /C16: track 293.6 -> 432.4 mm, vias 7 -> 6
- net /C15: track 287.4 -> 419.8 mm, vias 7 -> 6
- net /C14: track 262.0 -> 391.1 mm, vias 5 -> 4
- net /C12: track 247.8 -> 375.6 mm, vias 7 -> 6
- net /C11: track 227.9 -> 354.9 mm, vias 7 -> 6
- net /C10: track 208.2 -> 334.9 mm, vias 7 -> 6
- net /VOL: track 143.6 -> 30.8 mm, vias 3 -> 2
- net VBUS: track 0.00 -> 108.2 mm, vias 0 -> 26
- net /C6: track 130.2 -> 229.5 mm, vias 7 -> 6
- net VDD: track 12.1 -> 110.7 mm, vias 6 -> 3
- net /TERMINAL_A: track 178.0 -> 82.7 mm, vias 4 -> 0
- net /TERMINAL_B: track 177.1 -> 82.3 mm, vias 4 -> 0
- net /LED_DATA: track 154.8 -> 60.2 mm, vias 2 -> 0
- net /SW: track 169.2 -> 74.9 mm, vias 2 -> 0
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- added copper zone on B.Cu, net VBUS
- added copper zone on F.Cu, net VBUS
- removed copper zone on B.Cu, net +5V
- removed copper zone on F.Cu, net +5V
- removed copper zone on F.Cu, net VDD
Other:
- outline, holes or cut-outs redrawn
- board text added: "BOOT"
- board text added: "EN"
