File: MCU.kicad_sch (KiCad schematic)
At the start: 34 parts, among them J1 USB_C_Receptacle_USB2.0_16P, SW1 SW_Push, SW2 SW_Push, U1 RP2040, U2 W25Q128JVS, Y1 Crystal_GND24

Commit message: Finished V0.1
Parts:
- removed D91: 1N4148W, Diode_SMD:D_SOD-123, symbol Diode:1N4148W
- removed JP1: SolderJumper_3_Open, Jumper:SolderJumper-3_P1.3mm_Open_Pad1.0x1.5mm, symbol Jumper:SolderJumper_3_Open
- added TP19, TP20: TestPoint, TestPoint:TestPoint_Pad_D1.0mm, symbol Connector:TestPoint
Connections:
- net TESTEN is gone; now on net GND: U1.19 (TESTEN)
- net +3V3: now also TP1.1
- net USB_D+: now also TP20.1
- net USB_D-: now also TP19.1
- net C1 renamed IO11
- net C10 renamed IO4
- net C11 renamed IO5
- net C12 renamed IO6
- net C13 renamed IO7
- net C14 renamed IO8
- net C15 renamed IO9
- net C16 renamed IO10
- net C2 renamed IO12
- net C3 renamed IO13
- net C4 renamed IO14
- net C5 renamed IO15
- net C6 renamed IO0
- net C7 renamed IO1
- net C8 renamed IO2
- net C9 renamed IO3
- net R1 renamed IO16
- net R2 renamed IO17
- net R3 renamed IO21
- net R4 renamed IO20
- net R5 renamed IO19
- net R6 renamed IO18
Other:
- moved on the sheet: C11, C12, C13, C14, C2, C3, F1, J1, R1, R2, R3, R4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

Commit message: Updated main board + daughterboard layout - V0.3
Parts:
- removed U2: W25Q128JVS, Package_SO:SOIC-8_5.3x5.3mm_P1.27mm, symbol Memory_Flash:W25Q128JVS
- added C23, C24: 10uF, Capacitor_SMD:C_0805_2012Metric, symbol Device:C
- added U2: NCP1117-3.3_SOT223, Package_TO_SOT_SMD:SOT-223-3_TabPin2, symbol Regulator_Linear:NCP1117-3.3_SOT223
- added U3: W25Q128JVE, Package_SON:WSON-8-1EP_8x6mm_P1.27mm_EP3.4x4.3mm, symbol Memory_Flash:W25Q128JVE
- C1, C11, C12, C16: footprint Capacitor_SMD:C_0402_1005Metric_Pad0.74x0.62mm_HandSolder -> Capacitor_SMD:C_0402_1005Metric
- C10, C13, C14, C2, C3, C4, C5, C6, C7, C8, C9: value 100nF -> 0.1uF; footprint Capacitor_SMD:C_0402_1005Metric_Pad0.74x0.62mm_HandSolder -> Capacitor_SMD:C_0402_1005Metric
- R1, R2, R4, R5, R8: footprint Resistor_SMD:R_0603_1608Metric_Pad0.98x0.95mm_HandSolder -> Resistor_SMD:R_0603_1608Metric
- R3: footprint Resistor_SMD:R_0603_1608Metric_Pad0.98x0.95mm_HandSolder -> Resistor_SMD:R_0402_1005Metric
- U1: footprint Package_DFN_QFN:QFN-56-1EP_7x7mm_P0.4mm_EP3.2x3.2mm -> Package_DFN_QFN:QFN-56-1EP_7x7mm_P0.4mm_EP3.2x3.2mm_ThermalVias
- Y1: footprint Crystal:Crystal_SMD_3225-4Pin_3.2x2.5mm_HandSoldering -> Crystal:Crystal_SMD_3225-4Pin_3.2x2.5mm
Connections:
- net +3V3: now also U3.8 (VCC)
- net GND: now also C23.2, C24.2, U2.1 (GND), U3.4 (GND), U3.9 (EP)
- net QSPI_SCLK: now also U3.6 (CLK)
- net QSPI_SD0: now also U3.5 (DI/IO_{0})
- net QSPI_SD1: now also U3.2 (DO/IO_{1})
- net QSPI_SD2: now also U3.3 (~{WP}/IO_{2})
- net QSPI_SD3: now also U3.7 (~{HOLD}/~{RESET}/IO_{3})
- net QSPI_SS: now also U3.1 (~{CS})
- net SWCLK: now also TP3.1; no longer TP2.1
- net SWD: now also TP2.1; no longer TP3.1
- net VDD: now also J1.A5 (CC1), J1.B5 (CC2), C24.1, U2.2 (VO); no longer J1.A4 (VBUS), J1.A9 (VBUS), J1.B4 (VBUS), J1.B9 (VBUS)
- net EN: no longer names the net of C14.2, R8.2, SW2.2, U1.26 (RUN)
- new net VBUS: C23.1, J1.A4 (VBUS), J1.A9 (VBUS), J1.B4 (VBUS), J1.B9 (VBUS), U2.3 (VI)
- no-connect marks 4 -> 2
Other:
- moved on the sheet: F1
