File: nes_keyboard.kicad_sch (KiCad schematic)
At the start: 209 parts, among them J2 Conn_01x02_Pin, SW3 RotaryEncoder_Switch_MP, U4 74AHCT1G125

Commit message: Finished V0.1
Parts:
- added H1, H2, H3, H4, H5, H6, H7, H8, H9: MountingHole, MountingHole:MountingHole_2.2mm_M2, symbol Mechanical:MountingHole
- added TP18: TestPoint, TestPoint:TestPoint_Pad_D1.0mm, symbol Connector:TestPoint
- R13: value R -> 100
- SW3: footprint Rotary_Encoder:RotaryEncoder_Alps_EC11E-Switch_Vertical_H20mm -> Rotary_Encoder:RotaryEncoder_Bourns_Vertical_PEC12R-3x17F-Sxxxx
Connections:
- net +5V: now also TP18.1
Other:
- sheet MCU ports: added IO0, IO1, IO10, IO11, IO12, IO13, IO14, IO15, IO16, IO17, IO18, IO19, IO2, IO20, IO21, IO3, IO4, IO5, IO6, IO7, IO8, IO9; removed C1, C10, C11, C12, C13, C14, C15, C16, C2, C3, C4, C5, C6, C7, C8, C9, R1, R2, R3, R4, R5, R6
- moved on the sheet: C15, C17, C18, C19, C20, C21, C22, C25, C26, C27, C28, C29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

Commit message: Updated main board + daughterboard layout - V0.3
Parts:
- removed J2: Conn_01x02_Pin, Connector_Hirose:Hirose_DF13-02P-1.25DS_1x02_P1.25mm_Horizontal, symbol Connector:Conn_01x02_Pin
- removed TP17, TP18: TestPoint, TestPoint:TestPoint_Pad_D1.0mm, symbol Connector:TestPoint
- added S85, S86, S87: Keyswitch, PCM_Mounting_Keyboard_Stabilizer:Stabilizer_Cherry_MX_2.00u, symbol ScottoKeebs:Placeholder_Keyswitch
- added S88: Keyswitch, PCM_Mounting_Keyboard_Stabilizer:Stabilizer_Cherry_MX_6.25u, symbol ScottoKeebs:Placeholder_Keyswitch
- C15: footprint Capacitor_SMD:C_0603_1608Metric_Pad1.08x0.95mm_HandSolder -> Capacitor_SMD:C_0805_2012Metric
- C17, C18, C19, C20, C21, C22: footprint Capacitor_SMD:C_0603_1608Metric_Pad1.08x0.95mm_HandSolder -> Capacitor_SMD:C_0603_1608Metric
- C25, C26, C27, C28, C29: footprint Capacitor_SMD:C_0402_1005Metric_Pad0.74x0.62mm_HandSolder -> Capacitor_SMD:C_0402_1005Metric
- R10, R11, R12, R7, R9: footprint Resistor_SMD:R_0402_1005Metric_Pad0.72x0.64mm_HandSolder -> Resistor_SMD:R_0402_1005Metric
- R13: footprint Resistor_SMD:R_0603_1608Metric_Pad0.98x0.95mm_HandSolder -> Resistor_SMD:R_0603_1608Metric
Connections:
- net +5V renamed VBUS
