File: nes_keyboard_daughterboard/nes_keyboard_daughterboard.kicad_sch (KiCad schematic)
At the start: 17 parts, among them J1 USB_C_Receptacle_USB2.0_16P, J2 Conn_01x02_Pin, J3 USB_C_Receptacle_USB2.0_16P, U1 NCP1117-3.3_SOT223, U2 USBLC6-2P6

Commit message: Finished V0.1
Parts:
- added V1: 5, symbol Simulation_SPICE:VDC
- R3: value 220 -> 680
- R4: value 130 -> 470
Connections:
- net GND: now also V1.2
- net VBUS: now also V1.1
Other:
- moved on the sheet: C1, C2, D1, H1, H2, H3, H4, J1, J2, J3, R1, R2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

Commit message: PCB Modifications (all) - V0.2
Parts:
- C1, C2: footprint Capacitor_SMD:C_0603_1608Metric_Pad1.08x0.95mm_HandSolder -> Capacitor_SMD:C_0805_2012Metric_Pad1.18x1.45mm_HandSolder; LCSC (none) -> C95841
- D1, D2: LCSC (none) -> C19171390
- J1: LCSC (none) -> C7095263
- J2: footprint Connector_Hirose:Hirose_DF13-02P-1.25DSA_1x02_P1.25mm_Vertical -> Connector_JST:JST_PH_S2B-PH-K_1x02_P2.00mm_Horizontal; LCSC (none) -> C17264620
- J3: LCSC (none) -> C3020560
- R1, R2: LCSC (none) -> C112314
- R3: LCSC (none) -> C112310
- R4: LCSC (none) -> C114433
- U1: LCSC (none) -> C26537
- U2: LCSC (none) -> C15999
Changed lines of the file:
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@@
 			)
 		)
+		(property "LCSC" ""
+			(at 130.81 128.27 0)
+			(hide yes)
+			(show_name no)
+			(do_not_autoplace no)
+			(effects
+				(font
+					(size 1.27 1.27)
+				)
+			)
+		)
 		(pin "1"
 		)
@@
 			)
 		)
-		(property "Footprint" "Connector_Hirose:Hirose_DF13-02P-1.25DSA_1x02_P1.25mm_Vertical"
+		(property "Footprint" "Connector_JST:JST_PH_S2B-PH-K_1x02_P2.00mm_Horizontal"
 			(at 87.63 121.92 0)
 			(hide yes)
@@
 			)
 		)
+		(property "LCSC" "C17264620"
+			(at 87.63 121.92 0)
+			(hide yes)
+			(show_name no)
+			(do_not_autoplace no)
+			(effects
+				(font
+					(size 1.27 1.27)
+				)
+			)
+		)
 		(pin "1"
 		)
@@
 			)
 		)
+		(property "LCSC" "C19171390"
+			(at 213.36 52.07 90)
+			(hide yes)
+			(show_name no)
+			(do_not_autoplace no)
+			(effects
+				(font
+					(size 1.27 1.27)
+				)
+			)
+		)
 		(pin "1"
 		)
@@
 			)
 		)
+		(property "LCSC" ""
+			(at 130.81 113.03 0)
+			(hide yes)
+			(show_name no)
+			(do_not_autoplace no)
+			(effects
+				(font
+					(size 1.27 1.27)
+				)
+			)
+		)
 		(pin "1"
 		)
@@
 			)
 		)
-		(property "Footprint" "Capacitor_SMD:C_0603_1608Metric_Pad1.08x0.95mm_HandSolder"
+		(property "Footprint" "Capacitor_SMD:C_0805_2012Metric_Pad1.18x1.45mm_HandSolder"
 			(at 148.8948 54.61 0)
 			(hide yes)
@@
 			)
 		)
+		(property "LCSC" "C95841"
+			(at 149.86 58.42 0)
+			(hide yes)
+			(show_name no)
+			(do_not_autoplace no)
+			(effects
+				(font
+					(size 1.27 1.27)
+				)
+			)
+		)
 		(pin "1"
 		)
@@
 			)
 		)
+		(property "LCSC" "C3020560"
+			(at 48.26 121.92 0)
+			(hide yes)
+			(show_name no)
+			(do_not_autoplace no)
+			(effects
+				(font
+					(size 1.27 1.27)
+				)
+			)
+		)
 		(pin "B1"
 		)
@@
 			)
 		)
+		(property "LCSC" "C112314"
+			(at 68.58 48.26 90)
+			(hide yes)
+			(show_name no)
+			(do_not_autoplace no)
+			(effects
+				(font
+					(size 1.27 1.27)
+				)
+			)
+		)
 		(pin "1"
 		)
@@
 			)
 		)
+		(property "LCSC" "C19171390"
+			(at 198.12 52.07 90)
+			(hide yes)
+			(show_name no)
+			(do_not_autoplace no)
+			(effects
+				(font
+					(size 1.27 1.27)
+				)
+			)
+		)
 		(pin "1"
 		)
@@
 			)
 		)
+		(property "LCSC" "C26537"
+			(at 162.56 53.34 0)
+			(hide yes)
+			(show_name no)
+			(do_not_autoplace no)
+			(effects
+				(font
+					(size 1.27 1.27)
+				)
+			)
+		)
 		(pin "2"
 		)
@@
 			)
 		)
+		(property "LCSC" "C7095263"
+			(at 48.26 55.88 0)
+			(hide yes)
+			(show_name no)
+			(do_not_autoplace no)
+			(effects
+				(font
+					(size 1.27 1.27)
+				)
+			)
+		)
 		(pin "A4"
 		)
@@
 			)
 		)
+		(property "LCSC" "C112314"
+			(at 68.58 45.72 90)
+			(hide yes)
+			(show_name no)
+			(do_not_autoplace no)
+			(effects
+				(font
+					(size 1.27 1.27)
+				)
+			)
+		)
 		(pin "1"
 		)
@@
 			)
 		)
+		(property "LCSC" ""
+			(at 153.67 128.27 0)
+			(hide yes)
+			(show_name no)
+			(do_not_autoplace no)
+			(effects
+				(font
+					(size 1.27 1.27)
+				)
+			)
+		)
 		(pin "1"
 		)
@@
 			)
 		)
+		(property "LCSC" "C15999"
+			(at 102.87 57.15 0)
+			(hide yes)
+			(show_name no)
+			(do_not_autoplace no)
+			(effects
+				(font
+					(size 1.27 1.27)
+				)
+			)
+		)
 		(pin "1"
 		)
@@
 			)
 		)
+		(property "LCSC" ""
+			(at 205.74 123.19 0)
+			(hide yes)
+			(show_name no)
+			(do_not_autoplace no)
+			(effects
+				(font
+					(size 1.27 1.27)
+				)
+			)
+		)
 		(pin "2"
 		)
@@
 			)
 		)
+		(property "LCSC" "C112310"
+			(at 198.12 60.96 0)
+			(hide yes)
+			(show_name no)
+			(do_not_autoplace no)
+			(effects
+				(font
+					(size 1.27 1.27)
+				)
+			)
+		)
 		(pin "2"
 		)
@@
 			)
 		)
+		(property "LCSC" ""
+			(at 153.67 113.03 0)
+			(hide yes)
+			(show_name no)
+			(do_not_autoplace no)
+			(effects
+				(font
+					(size 1.27 1.27)
+				)
+			)
+		)
 		(pin "1"
 		)
@@
 			)
 		)
-		(property "Footprint" "Capacitor_SMD:C_0603_1608Metric_Pad1.08x0.95mm_HandSolder"
+		(property "Footprint" "Capacitor_SMD:C_0805_2012Metric_Pad1.18x1.45mm_HandSolder"
 			(at 174.2948 54.61 0)
 			(hide yes)
@@
 			)
 		)
+		(property "LCSC" "C95841"
+			(at 175.26 58.42 0)
+			(hide yes)
+			(show_name no)
+			(do_not_autoplace no)
+			(effects
+				(font
+					(size 1.27 1.27)
+				)
+			)
+		)
 		(pin "1"
 		)
@@
 			(at 213.36 60.96 0)
 			(hide yes)
+			(show_name no)
+			(do_not_autoplace no)
+			(effects
+				(font
+					(size 1.27 1.27)
+				)
+			)
+		)
+		(property "LCSC" "C114433"
+			(at 213.36 60.96 0)
+			(hide yes)

Commit message: Updated main board + daughterboard layout - V0.3
Parts:
- removed C1, C2: 10uF, Capacitor_SMD:C_0805_2012Metric_Pad1.18x1.45mm_HandSolder, symbol Device:C
- removed J2: Conn_01x02_Pin, Connector_JST:JST_PH_S2B-PH-K_1x02_P2.00mm_Horizontal, symbol Connector:Conn_01x02_Pin
- removed U1: NCP1117-3.3_SOT223, Package_TO_SOT_SMD:SOT-223-3_TabPin2, symbol Regulator_Linear:NCP1117-3.3_SOT223
- removed V1: 5, symbol Simulation_SPICE:VDC
Connections:
- net +3V3: now also J3.A5 (CC1), J3.B5 (CC2); no longer J3.A4 (VBUS), J3.A9 (VBUS), J3.B4 (VBUS), J3.B9 (VBUS)
- net VBUS: now also J3.A4 (VBUS), J3.A9 (VBUS), J3.B4 (VBUS), J3.B9 (VBUS)
- no-connect marks 6 -> 4
Other:
- moved on the sheet: D1, D2, H1, H2, H3, H4, J1, J3, R1, R2, R3, R4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

Commit message: Created and added 3D files - V0.5
Parts:
- added C1, C2: 10uF, Capacitor_SMD:C_0805_2012Metric, symbol Device:C
- added F1: 500mA, Fuse:Fuse_0603_1608Metric, symbol Device:Fuse
- added U1: NCP1117-3.3_SOT223, Package_TO_SOT_SMD:SOT-223-3_TabPin2, symbol Regulator_Linear:NCP1117-3.3_SOT223
- D1, D2: Digikey Link (none) -> https://www.digikey.ca/en/products/detail/liteon/LTST-C191K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; LCSC C19171390 -> (none); Part Num. (none) -> LTST-C191KRKT
- J1: Digikey Link (none) -> https://www.digikey.ca/en/products/detail/gct/USB4085-GF-A/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; LCSC C7095263 -> (none); Part Num. (none) -> USB4085-GF-A
- J3: Digikey Link (none) -> https://www.digikey.ca/en/products/detail/gct/USB4105-GF-A/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; LCSC C3020560 -> (none); Part Num. (none) -> USB4105-GF-A
- R1, R2: Digikey Link (none) -> https://www.digikey.ca/en/products/detail/yageo/RC0603FR-07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; LCSC C112314 -> (none); Part Num. (none) -> RC0603FR-075K1L
- R3: Digikey Link (none) -> https://www.digikey.ca/en/products/detail/yageo/RC0603JR-07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; LCSC C112310 -> (none); Part Num. (none) -> RC0603JR-07680RL
- R4: Digikey Link (none) -> https://www.digikey.ca/en/products/detail/te-connectivity-p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; LCSC C114433 -> (none); Part Num. (none) -> CRGCQ0603F470R
- U2: Digikey Link (none) -> https://www.digikey.ca/en/products/detail/stmicroelectronic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; LCSC C15999 -> (none); Part Num. (none) -> USBLC6-2P6
Connections:
- net +3V3: now also J3.A4 (VBUS), J3.A9 (VBUS), J3.B4 (VBUS), J3.B9 (VBUS), F1.2; no longer D2.2 (A), J3.A5 (CC1), J3.B5 (CC2)
- net GND: now also C1.2, C2.2, U1.1 (GND); no longer J1.S1 (SHIELD), J3.S1 (SHIELD)
- net VBUS: now also J3.A5 (CC1), J3.B5 (CC2), C1.1, U1.3 (VI); no longer J3.A4 (VBUS), J3.A9 (VBUS), J3.B4 (VBUS), J3.B9 (VBUS)
- new net VDD: C2.1, D2.2 (A), F1.1, U1.2 (VO)
- no-connect marks 4 -> 6
