File: nes_switchplate/nes_switchplate.kicad_pcb (KiCad board)
At the start: 2 copper layers, 323.9 x 115.5 mm, 9 parts

Commit message: Created and added 3D files - V0.5
Parts:
- moved H4 47.5 mm to (111.0, 17.0)
- moved H6 47.5 mm to (190.5, 17.0)
- moved H8 47.5 mm to (266.7, 17.0)
- moved H1 47.5 mm to (57.2, 17.0)
- moved H3 47.5 mm to (59.0, 80.3)
- moved H7 47.5 mm to (223.9, 74.1)
- moved H9 47.5 mm to (282.0, 83.2)
- moved H2 47.5 mm to (19.1, 44.4)
- moved H5 47.5 mm to (147.7, 74.1)
Other:
- board size 323.9 x 115.5 mm -> 325 x 116.5 mm
