File: nes_switchplate/nes_switchplate.kicad_pcb (KiCad board)
At the start: 2 copper layers, 325 x 116.5 mm, 9 parts

Commit message: Fixed footprints, created firmware - V1
Changed lines of the file:
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@@
 			(at 0 -3.15 0)
 			(layer "F.SilkS")
+			(hide yes)
 			(effects
 				(font
@@
 		(layer "Dwgs.User")
 		(pts
-			(xy 2 -2) (xy 2.002482 113.5)
+			(xy 0.430001 -2.5) (xy 0.43 114)
 		)
 		(height -17)
@@
 			(keep_text_aligned yes)
 		)
-		(gr_text "115.5"
-			(at -16.15 55.75 90)
+		(gr_text "116.5"
+			(at -17.719999 55.75 90)
 			(layer "Dwgs.User")
 			(effects
@@
 		(layer "Dwgs.User")
 		(pts
-			(xy 0 0) (xy 323.866077 1.046627)
+			(xy -0.57 -1.5) (xy 324.438514 -1.5)
 		)
 		(height -24.35)
@@
 			(keep_text_aligned yes)
 		)
-		(gr_text "323.8661"
-			(at 161.933039 -25.5 0)
+		(gr_text "325.0085"
+			(at 161.934257 -27 0)
 			(layer "Dwgs.User")
 			(effects
