File: nes_switchplate/nes_switchplate.kicad_sch (KiCad schematic)
At the start: 0 parts

Commit message: Created and added 3D files - V0.5
Parts:
- added H1, H2, H3, H4, H5, H6, H7, H8, H9: MountingHole, MountingHole:MountingHole_2.2mm_M2, symbol Mechanical:MountingHole
