File: nes_mainboard/MCU.kicad_sch (KiCad schematic)
At the start: 33 parts, among them J1 USB_C_Receptacle_USB2.0_16P, SW1 SW_Push, SW2 SW_Push, U1 RP2040, U3 W25Q128JVE, Y1 Crystal_GND24

Commit message: Fixed footprints, created firmware - V1
Parts:
- R4: value R -> 1k; Digikey Link (none) -> https://www.digikey.ca/en/products/detail/yageo/RC0603FR-07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; Part Num. (none) -> RC0603FR-071KL; now fitted; now in the parts list
- R5: value 1k -> 0; Digikey Link https://www.digikey.ca/en/products/detail/yageo/RC0603FR-07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 -> (none); Part Num. RC0603FR-071KL -> (none)
- U1: footprint Package_DFN_QFN:QFN-56-1EP_7x7mm_P0.4mm_EP3.2x3.2mm_ThermalVias -> Package_DFN_QFN:QFN-56-1EP_7x7mm_P0.4mm_EP3.2x3.2mm
Connections:
- net QSPI_SS: no longer R4.2, R5.2, U3.1 (~{CS})
- new net ~{QSPI_SS}: R4.2, R5.2, U3.1 (~{CS})
Changed lines of the file:
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@@
 		)
 	)
-	(label "QSPI_SS"
+	(label "~{QSPI_SS}"
 		(at 139.7 110.49 0)
 		(effects
@@
 			)
 		)
-		(property "Value" "1k"
+		(property "Value" "0"
 			(at 133.35 110.49 90)
 			(show_name no)
@@
 			)
 		)
-		(property "Digikey Link" "https://www.digikey.ca/en/products/detail/yageo/RC0603FR-071KL/726843"
+		(property "Digikey Link" ""
 			(at 133.35 110.49 90)
 			(hide yes)
@@
 			)
 		)
-		(property "Part Num." "RC0603FR-071KL"
+		(property "Part Num." ""
 			(at 133.35 110.49 90)
 			(hide yes)
@@
 			)
 		)
-		(property "Footprint" "Package_DFN_QFN:QFN-56-1EP_7x7mm_P0.4mm_EP3.2x3.2mm_ThermalVias"
+		(property "Footprint" "Package_DFN_QFN:QFN-56-1EP_7x7mm_P0.4mm_EP3.2x3.2mm"
 			(at 74.93 96.52 0)
 			(hide yes)
@@
 		(body_style 1)
 		(exclude_from_sim no)
-		(in_bom no)
+		(in_bom yes)
 		(on_board yes)
 		(in_pos_files yes)
-		(dnp yes)
+		(dnp no)
 		(fields_autoplaced yes)
 		(property "Reference" "R4"
@@
 			)
 		)
-		(property "Value" "R"
+		(property "Value" "1k"
 			(at 140.97 102.8699 0)
 			(show_name no)
@@
 			(at 138.43 101.6 0)
 			(hide yes)
+			(show_name no)
+			(do_not_autoplace no)
+			(effects
+				(font
+					(size 1.27 1.27)
+				)
+			)
+		)
+		(property "Digikey Link" "https://www.digikey.ca/en/products/detail/yageo/RC0603FR-071KL/726843"
+			(at 138.43 101.6 0)
+			(hide yes)
+			(show_name no)
+			(do_not_autoplace no)
+			(effects
+				(font
+					(size 1.27 1.27)
+				)
+			)
+		)
+		(property "Part Num." "RC0603FR-071KL"
+			(at 138.43 101.6 0)
+			(hide yes)
