File: nes_mainboard/nes_keyboard.kicad_pcb (KiCad board)
At the start: 2 copper layers, 323.9 x 115.5 mm, 253 parts, among them J1 USB_C_Receptacle_USB2.0_16P, SW1 SW_Push, SW2 SW_Push, SW3 RotaryEncoder_Switch_MP, U1 RP2040, U3 W25Q128JVE, U4 74AHCT1G125, Y1 Crystal_GND24

Commit message: Fixed footprints, created firmware - V1
Parts:
- added TP17: TestPoint, TestPoint:TestPoint_Pad_D1.0mm, F.Cu at (72.4, 140.8)
- added TP18: TestPoint, TestPoint:TestPoint_Pad_D1.0mm, F.Cu at (72.0, 145.4)
- R4: value R -> 1k
- R5: value 1k -> 0
- U1: footprint Package_DFN_QFN:QFN-56-1EP_7x7mm_P0.4mm_EP3.2x3.2mm_ThermalVias -> Package_DFN_QFN:QFN-56-1EP_7x7mm_P0.4mm_EP3.2x3.2mm
Connections:
- R4 pad 2: /MCU/QSPI_SS -> /MCU/~{QSPI_SS}
- R5 pad 2: /MCU/QSPI_SS -> /MCU/~{QSPI_SS}
- U3 pad 1: /MCU/QSPI_SS -> /MCU/~{QSPI_SS}
Routing:
- net Net-(D85-DOUT): track 19.2 -> 0.00 mm
- net Net-(D88-DOUT): track 19.2 -> 0.00 mm
- net Net-(D87-DOUT): track 19.2 -> 0.00 mm
- net Net-(D86-DOUT): track 19.2 -> 0.00 mm
- net Net-(D89-DOUT): track 11.0 -> 0.00 mm
- net /D_REG: track 6.40 -> 4.08 mm
- net GND: vias 54 -> 58
