File: nes_mainboard/nes_keyboard.kicad_sch (KiCad schematic)
At the start: 220 parts, among them SW3 RotaryEncoder_Switch_MP, U4 74AHCT1G125

Commit message: Fixed footprints, created firmware - V1
Parts:
- added TP17, TP18: TestPoint, TestPoint:TestPoint_Pad_D1.0mm, symbol Connector:TestPoint
Connections:
- net +3V3: now also TP17.1
- net VBUS: now also TP18.1
- no-connect marks 1 -> 4
